File: AmiPET.kicad_sch (KiCad schematic)
At the start: 9 parts, among them J1 Power, J2 Digital/PWM, J3 Analog, J4 Digital/PWM, J5 AMIGA Keyboard, J6 PET Keyboard Connector, J7 AMIGA Keyboard Connector, J8 PET Keyboard, U1 M3493B2

Commit message: PCB Project update
tweaked layout
new 3d models
added schematic, production files, bom and image
removed old painted schematic
Parts:
- added C1: C, Capacitor_THT:C_Disc_D6.0mm_W2.5mm_P5.00mm, symbol Device:C
- J1, J4: footprint Connector_PinSocket_2.54mm:PinSocket_1x08_P2.54mm_Vertical -> AmiPet_lib_fp:PinSocket_1x08_P2.54mm_Vertical
- J2: footprint Connector_PinSocket_2.54mm:PinSocket_1x10_P2.54mm_Vertical -> AmiPet_lib_fp:PinSocket_1x10_P2.54mm_Vertical
- J3: footprint Connector_PinSocket_2.54mm:PinSocket_1x06_P2.54mm_Vertical -> AmiPet_lib_fp:PinSocket_1x06_P2.54mm_Vertical
- J6: symbol Connector:Conn_01x20_Male -> Connector:Conn_01x20_Pin
- J7: symbol Connector:Conn_01x04_Male -> Connector:Conn_01x04_Pin
- J8: symbol Connector:Conn_01x20_Female -> Connector:Conn_01x20_Socket
Connections:
- net GND: now also C1.2
- net VCC: now also C1.1
